File: ITX-Mainboard/Wrap030-ITX/IRQ.kicad_sch (KiCad schematic)
At the start: 10 parts, among them U32 ATF1508AS

Commit message: Completing PCB Routing
Parts:
- removed C1 (x3): 100nF, Capacitor_SMD:C_0402_1005Metric_Pad0.74x0.62mm_HandSolder, symbol Device:C_Small
Other:
- company: (none) -> techav
- title: (none) -> Wrap030-ATX Mainboard

Commit message: Replace resistor nets with 0402 & update gerbers
Parts:
- C1: Mouser-Part (none) -> 187-CL05B104KO5NNNC; Notes (none) -> JLC
- C15: Mouser-Part (none) -> 187-CL05A105KA5NQNC; Notes (none) -> JLC
- U32: Mouser-Part (none) -> 556-ATF1508AS-10JU84; Notes (none) -> OFE; Socket-Mouser (none) -> 575-948424
Changed lines of the file:
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@@
       (effects (font (size 1.27 1.27)) hide)
     )
-    (property "Mouser-Part" "" (at 144.78 104.14 0)
-      (effects (font (size 1.27 1.27)) hide)
-    )
-    (property "Notes" "" (at 144.78 104.14 0)
+    (property "Mouser-Part" "187-CL05B104KO5NNNC" (at 144.78 104.14 0)
+      (effects (font (size 1.27 1.27)) hide)
+    )
+    (property "Notes" "JLC" (at 144.78 104.14 0)
+      (effects (font (size 1.27 1.27)) hide)
+    )
+    (property "Socket-Mouser" "" (at 144.78 104.14 0)
       (effects (font (size 1.27 1.27)) hide)
     )
@@
     )
     (property "Datasheet" "" (at 76.2 50.8 0)
+      (effects (font (size 1.27 1.27)) hide)
+    )
+    (property "Mouser-Part" "556-ATF1508AS-10JU84" (at 76.2 50.8 0)
+      (effects (font (size 1.27 1.27)) hide)
+    )
+    (property "Notes" "OFE" (at 76.2 50.8 0)
+      (effects (font (size 1.27 1.27)) hide)
+    )
+    (property "Socket-Mouser" "575-948424" (at 76.2 50.8 0)
       (effects (font (size 1.27 1.27)) hide)
     )
@@
       (effects (font (size 1.27 1.27)) hide)
     )
-    (property "Mouser-Part" "" (at 160.02 104.14 0)
-      (effects (font (size 1.27 1.27)) hide)
-    )
-    (property "Notes" "" (at 160.02 104.14 0)
+    (property "Mouser-Part" "187-CL05B104KO5NNNC" (at 160.02 104.14 0)
+      (effects (font (size 1.27 1.27)) hide)
+    )
+    (property "Notes" "JLC" (at 160.02 104.14 0)
+      (effects (font (size 1.27 1.27)) hide)
+    )
+    (property "Socket-Mouser" "" (at 160.02 104.14 0)
       (effects (font (size 1.27 1.27)) hide)
     )
@@
     )
     (property "Datasheet" "" (at 165.1 63.5 0)
+      (effects (font (size 1.27 1.27)) hide)
+    )
+    (property "Mouser-Part" "556-ATF1508AS-10JU84" (at 165.1 63.5 0)
+      (effects (font (size 1.27 1.27)) hide)
+    )
+    (property "Notes" "OFE" (at 165.1 63.5 0)
+      (effects (font (size 1.27 1.27)) hide)
+    )
+    (property "Socket-Mouser" "575-948424" (at 165.1 63.5 0)
       (effects (font (size 1.27 1.27)) hide)
     )
@@
       (effects (font (size 1.27 1.27)) hide)
     )
-    (property "Mouser-Part" "" (at 149.86 104.14 0)
-      (effects (font (size 1.27 1.27)) hide)
-    )
-    (property "Notes" "" (at 149.86 104.14 0)
+    (property "Mouser-Part" "187-CL05B104KO5NNNC" (at 149.86 104.14 0)
+      (effects (font (size 1.27 1.27)) hide)
+    )
+    (property "Notes" "JLC" (at 149.86 104.14 0)
+      (effects (font (size 1.27 1.27)) hide)
+    )
+    (property "Socket-Mouser" "" (at 149.86 104.14 0)
       (effects (font (size 1.27 1.27)) hide)
     )
@@
       (effects (font (size 1.27 1.27)) hide)
     )
-    (property "Mouser-Part" "" (at 165.1 104.14 0)
-      (effects (font (size 1.27 1.27)) hide)
-    )
-    (property "Notes" "" (at 165.1 104.14 0)
+    (property "Mouser-Part" "187-CL05B104KO5NNNC" (at 165.1 104.14 0)
+      (effects (font (size 1.27 1.27)) hide)
+    )
+    (property "Notes" "JLC" (at 165.1 104.14 0)
+      (effects (font (size 1.27 1.27)) hide)
+    )
+    (property "Socket-Mouser" "" (at 165.1 104.14 0)
       (effects (font (size 1.27 1.27)) hide)
     )
@@
       (effects (font (size 1.27 1.27)) hide)
     )
-    (property "Mouser-Part" "" (at 139.7 104.14 0)
-      (effects (font (size 1.27 1.27)) hide)
-    )
-    (property "Notes" "" (at 139.7 104.14 0)
+    (property "Mouser-Part" "187-CL05A105KA5NQNC" (at 139.7 104.14 0)
+      (effects (font (size 1.27 1.27)) hide)
+    )
+    (property "Notes" "JLC" (at 139.7 104.14 0)
+      (effects (font (size 1.27 1.27)) hide)
+    )
+    (property "Socket-Mouser" "" (at 139.7 104.14 0)
       (effects (font (size 1.27 1.27)) hide)
     )
@@
       (effects (font (size 1.27 1.27)) hide)
     )
-    (property "Mouser-Part" "" (at 154.94 104.14 0)
-      (effects (font (size 1.27 1.27)) hide)
-    )
-    (property "Notes" "" (at 154.94 104.14 0)
-      (effects (font (size 1.27 1.27)) hide)
-    )
+    (property "Mouser-Part" "187-CL05B104KO5NNNC" (at 154.94 104.14 0)
+      (effects (font (size 1.27 1.27)) hide)
+    )
+    (property "Notes" "JLC" (at 154.94 104.14 0)
+      (effects (font (size 1.27 1.27)) hide)
+    )
+    (property "Socket-Mouser" "" (at 154.94 104.14 0)
+      (effects (font (size 1.27 1.27)) hide)
+    )
