File: ITX-Mainboard/Wrap030-ITX/ISA-IDE-Con.kicad_sch (KiCad schematic)
At the start: 6 parts, among them J10 Conn_02x20_Odd_Even, J4 Bus_ISA_16bit

Commit message: PCB substantial completion
Connections:
- net IDE-KEY: now reaches J10.20 (Pin_20)
Changed lines of the file:
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@@
+    (stroke (width 0) (type default))
+  )
+  (wire (pts (xy 69.85 176.53) (xy 82.55 176.53))
     (stroke (width 0) (type default))
   )
@@
     (stroke (width 0) (type default))
   )
+  (label "IDE-KEY" (at 82.55 176.53 180) (fields_autoplaced)
+    (effects (font (size 1.27 1.27)) (justify right bottom))
+  )
   (label "ISA-LA19" (at 165.1 114.3 180) (fields_autoplaced)

Commit message: Add interrupt controller to schematic
Connections:
- net ISA-IRQ7: now reaches J4.21 (IRQ7)
- net ISA-IRQ7: now also J4.21 (IRQ7), J4.21 (IRQ7)
- net ISA-IRQ6: now reaches J4.22 (IRQ6)
- net ISA-IRQ6: now also J4.22 (IRQ6), J4.22 (IRQ6)
- net ISA-IRQ5: now reaches J4.23 (IRQ5)
- net ISA-IRQ5: now also J4.23 (IRQ5), J4.23 (IRQ5)
- net ISA-IRQ4: now reaches J4.24 (IRQ4)
- net ISA-IRQ4: now also J4.24 (IRQ4), J4.24 (IRQ4)
- net ISA-IRQ3: now reaches J4.25 (IRQ3)
- net ISA-IRQ3: now also J4.25 (IRQ3), J4.25 (IRQ3)
- net ISA-IRQ2: now reaches J4.4 (IRQ2)
- net ISA-IRQ2: now also J4.4 (IRQ2), J4.4 (IRQ2)
- net ISA-IRQ10: now reaches J4.65 (IRQ10)
- net ISA-IRQ10: now also J4.65 (IRQ10), J4.65 (IRQ10)
- net ISA-IRQ11: now reaches J4.66 (IRQ11)
- net ISA-IRQ11: now also J4.66 (IRQ11), J4.66 (IRQ11)
- net ISA-IRQ12: now reaches J4.67 (IRQ12)
- net ISA-IRQ12: now also J4.67 (IRQ12), J4.67 (IRQ12)
- net ISA-IRQ15: now reaches J4.68 (IRQ15)
- net ISA-IRQ15: now also J4.68 (IRQ15), J4.68 (IRQ15)
- net ISA-IRQ14: now reaches J4.69 (IRQ14)
- net ISA-IRQ14: now also J4.69 (IRQ14), J4.69 (IRQ14)

Commit message: Completing PCB Routing
Other:
- title: Wrap030 ITX -> Wrap030-ATX Mainboard
Changed lines of the file:
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@@
   (paper "USLetter")
   (title_block
-    (title "Wrap030 ITX")
-    (date "2023-03-15")
-    (rev "0")
+    (title "Wrap030-ATX Mainboard")
+    (date "2023-03-26")
+    (rev "1")
     (company "techav")
   )

Commit message: initial production schematic
Parts:
- R1, R2: JLC-Part (none) -> https://jlcpcb.com/partdetail/18102-0805W8F1002T5E/C17414
Changed lines of the file:
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@@
       (effects (font (size 1.27 1.27)) hide)
     )
-    (property "JLC-Part" "" (at 38.1 189.23 0)
+    (property "JLC-Part" "https://jlcpcb.com/partdetail/18102-0805W8F1002T5E/C17414" (at 38.1 189.23 0)
       (effects (font (size 1.27 1.27)) hide)
     )
@@
       (effects (font (size 1.27 1.27)) hide)
     )
-    (property "JLC-Part" "" (at 38.1 186.69 0)
+    (property "JLC-Part" "https://jlcpcb.com/partdetail/18102-0805W8F1002T5E/C17414" (at 38.1 186.69 0)
       (effects (font (size 1.27 1.27)) hide)
     )

Commit message: Replace resistor nets with 0402 & update gerbers
Parts:
- J10: Mouser-Part (none) -> 710-61203921621; Notes (none) -> OFE
- J4: Mouser-Part (none) -> 571-5645169-4; Notes (none) -> eBay
- R1, R2: footprint Resistor_SMD:R_0805_2012Metric -> Resistor_SMD:R_0402_1005Metric_Pad0.72x0.64mm_HandSolder; JLC-Part https://jlcpcb.com/partdetail/18102-0805W8F1002T5E/C17414 -> https://jlcpcb.com/partdetail/26487-0402WGF1002TCE/C25744; Mouser-Part (none) -> 303-0402WGF1002TCE; Notes (none) -> JLC
Changed lines of the file:
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@@
+    )
+  )
+  (symbol (lib_id "Device:R_Small_US") (at 38.1 186.69 90) (unit 1)
+    (in_bom yes) (on_board yes) (dnp no)
+    (property "Reference" "R1" (at 34.29 187.96 90)
+      (effects (font (size 1.27 1.27)))
+    )
+    (property "Value" "10k" (at 41.91 187.96 90)
+      (effects (font (size 1.27 1.27)))
+    )
+    (property "Footprint" "Resistor_SMD:R_0402_1005Metric_Pad0.72x0.64mm_HandSolder" (at 38.1 186.69 0)
+      (effects (font (size 1.27 1.27)) hide)
+    )
+    (property "Datasheet" "~" (at 38.1 186.69 0)
+      (effects (font (size 1.27 1.27)) hide)
+    )
+    (property "JLC-Part" "https://jlcpcb.com/partdetail/26487-0402WGF1002TCE/C25744" (at 38.1 186.69 0)
+      (effects (font (size 1.27 1.27)) hide)
+    )
+    (property "Mouser-Part" "303-0402WGF1002TCE" (at 38.1 186.69 0)
+      (effects (font (size 1.27 1.27)) hide)
+    )
+    (property "Notes" "JLC" (at 38.1 186.69 0)
+      (effects (font (size 1.27 1.27)) hide)
+    )
+    (property "Socket-Mouser" "" (at 38.1 186.69 0)
+      (effects (font (size 1.27 1.27)) hide)
+    )
+    (pin "1")
+    (pin "2")
+    (instances
+      (project "Wrap030-ITX"
+        (path "/911cb688-7d4c-4194-bbd3-2b645bd8d53c/253789b7-cae8-486b-a073-f8f34e01a47f/716ad3df-63c5-43f8-ad43-3095516fd8be"
+          (reference "R1") (unit 1)
+        )
+        (path "/911cb688-7d4c-4194-bbd3-2b645bd8d53c/daefa06e-0bcc-4cd3-a849-7c099c212056"
+          (reference "R3") (unit 1)
+        )
+      )
     )
   )
@@
       (effects (font (size 1.27 1.27)) hide)
     )
-    (property "Mouser-Part" "" (at 62.23 176.53 0)
-      (effects (font (size 1.27 1.27)) hide)
-    )
-    (property "Notes" "" (at 62.23 176.53 0)
+    (property "Mouser-Part" "710-61203921621" (at 62.23 176.53 0)
+      (effects (font (size 1.27 1.27)) hide)
+    )
+    (property "Notes" "OFE" (at 62.23 176.53 0)
+      (effects (font (size 1.27 1.27)) hide)
+    )
+    (property "Socket-Mouser" "" (at 62.23 176.53 0)
       (effects (font (size 1.27 1.27)) hide)
     )
@@
       (effects (font (size 1.27 1.27)) hide)
     )
-    (property "Mouser-Part" "" (at 198.12 83.82 0)
-      (effects (font (size 1.27 1.27)) hide)
-    )
-    (property "Notes" "" (at 198.12 83.82 0)
+    (property "Mouser-Part" "571-5645169-4" (at 198.12 83.82 0)
+      (effects (font (size 1.27 1.27)) hide)
+    )
+    (property "Notes" "eBay" (at 198.12 83.82 0)
+      (effects (font (size 1.27 1.27)) hide)
+    )
+    (property "Socket-Mouser" "" (at 198.12 83.82 0)
       (effects (font (size 1.27 1.27)) hide)
     )
@@
     )
   )
-  (symbol (lib_id "Device:R_Small_US") (at 38.1 189.23 90) (unit 1)
-    (in_bom yes) (on_board yes) (dnp no)
-    (property "Reference" "R2" (at 40.739 188.5489 90)
-      (effects (font (size 1.27 1.27)))
-    )
-    (property "Value" "10k" (at 34.29 188.5221 90)
-      (effects (font (size 1.27 1.27)))
-    )
-    (property "Footprint" "Resistor_SMD:R_0805_2012Metric" (at 38.1 189.23 0)
-      (effects (font (size 1.27 1.27)) hide)
-    )
-    (property "Datasheet" "~" (at 38.1 189.23 0)
-      (effects (font (size 1.27 1.27)) hide)
-    )
-    (property "JLC-Part" "https://jlcpcb.com/partdetail/18102-0805W8F1002T5E/C17414" (at 38.1 189.23 0)
-      (effects (font (size 1.27 1.27)) hide)
-    )
-    (property "Mouser-Part" "" (at 38.1 189.23 0)
-      (effects (font (size 1.27 1.27)) hide)
-    )
-    (property "Notes" "" (at 38.1 189.23 0)
-      (effects (font (size 1.27 1.27)) hide)
-    )
-    (pin "1")
-    (pin "2")
-    (instances
-      (project "Wrap030-ITX"
-        (path "/911cb688-7d4c-4194-bbd3-2b645bd8d53c/253789b7-cae8-486b-a073-f8f34e01a47f/716ad3df-63c5-43f8-ad43-3095516fd8be"
-          (reference "R2") (unit 1)
-        )
-      )
-    )
-  )
   (symbol (lib_id "power:VCC") (at 116.84 25.4 90) (unit 1)
     (in_bom yes) (on_board yes) (dnp no) (fields_autoplaced)
@@
     )
   )
-  (symbol (lib_id "Device:R_Small_US") (at 38.1 186.69 90) (unit 1)
-    (in_bom yes) (on_board yes) (dnp no)
-    (property "Reference" "R1" (at 40.739 186.0089 90)
-      (effects (font (size 1.27 1.27)))
-    )
-    (property "Value" "10k" (at 34.29 185.9821 90)
-      (effects (font (size 1.27 1.27)))
-    )
-    (property "Footprint" "Resistor_SMD:R_0805_2012Metric" (at 38.1 186.69 0)
-      (effects (font (size 1.27 1.27)) hide)
-    )
-    (property "Datasheet" "~" (at 38.1 186.69 0)
-      (effects (font (size 1.27 1.27)) hide)
-    )
-    (property "JLC-Part" "https://jlcpcb.com/partdetail/18102-0805W8F1002T5E/C17414" (at 38.1 186.69 0)
-      (effects (font (size 1.27 1.27)) hide)
-    )
-    (property "Mouser-Part" "" (at 38.1 186.69 0)
-      (effects (font (size 1.27 1.27)) hide)
-    )
-    (property "Notes" "" (at 38.1 186.69 0)
-      (effects (font (size 1.27 1.27)) hide)
-    )
-    (pin "1")
-    (pin "2")
-    (instances
-      (project "Wrap030-ITX"
-        (path "/911cb688-7d4c-4194-bbd3-2b645bd8d53c/253789b7-cae8-486b-a073-f8f34e01a47f/716ad3df-63c5-43f8-ad43-3095516fd8be"
-          (reference "R1") (unit 1)
-        )
-      )
-    )
-  )
   (symbol (lib_id "power:VCC") (at 180.34 91.44 90) (unit 1)
     (in_bom yes) (on_board yes) (dnp no) (fields_autoplaced)
@@
       (effects (font (size 1.27 1.27)) hide)
     )
-    (property "Mouser-Part" "" (at 134.62 83.82 0)
-      (effects (font (size 1.27 1.27)) hide)
-    )
-    (property "Notes" "" (at 134.62 83.82 0)
+    (property "Mouser-Part" "571-5645169-4" (at 134.62 83.82 0)
+      (effects (font (size 1.27 1.27)) hide)
+    )
+    (property "Notes" "eBay" (at 134.62 83.82 0)
+      (effects (font (size 1.27 1.27)) hide)
+    )
+    (property "Socket-Mouser" "" (at 134.62 83.82 0)
       (effects (font (size 1.27 1.27)) hide)
     )
@@
     )
   )
+  (symbol (lib_id "Device:R_Small_US") (at 38.1 189.23 90) (unit 1)
+    (in_bom yes) (on_board yes) (dnp no)
+    (property "Reference" "R2" (at 34.29 190.5 90)
+      (effects (font (size 1.27 1.27)))
+    )
+    (property "Value" "10k" (at 41.91 190.5 90)
+      (effects (font (size 1.27 1.27)))
+    )
+    (property "Footprint" "Resistor_SMD:R_0402_1005Metric_Pad0.72x0.64mm_HandSolder" (at 38.1 189.23 0)
+      (effects (font (size 1.27 1.27)) hide)
+    )
+    (property "Datasheet" "~" (at 38.1 189.23 0)
+      (effects (font (size 1.27 1.27)) hide)
+    )
+    (property "JLC-Part" "https://jlcpcb.com/partdetail/26487-0402WGF1002TCE/C25744" (at 38.1 189.23 0)
+      (effects (font (size 1.27 1.27)) hide)
+    )
+    (property "Mouser-Part" "303-0402WGF1002TCE" (at 38.1 189.23 0)
+      (effects (font (size 1.27 1.27)) hide)
+    )
+    (property "Notes" "JLC" (at 38.1 189.23 0)
+      (effects (font (size 1.27 1.27)) hide)
+    )
+    (property "Socket-Mouser" "" (at 38.1 189.23 0)
+      (effects (font (size 1.27 1.27)) hide)
+    )
+    (pin "1")
+    (pin "2")
+    (instances
+      (project "Wrap030-ITX"
+        (path "/911cb688-7d4c-4194-bbd3-2b645bd8d53c/253789b7-cae8-486b-a073-f8f34e01a47f/716ad3df-63c5-43f8-ad43-3095516fd8be"
+          (reference "R2") (unit 1)
+        )
+        (path "/911cb688-7d4c-4194-bbd3-2b645bd8d53c/daefa06e-0bcc-4cd3-a849-7c099c212056"
+          (reference "R3") (unit 1)
+        )
+      )
+    )
+  )
   (symbol (lib_id "power:GND") (at 82.55 189.23 90) (unit 1)
     (in_bom yes) (on_board yes) (dnp no) (fields_autoplaced)
@@
       (effects (font (size 1.27 1.27)) hide)
     )
-    (property "Mouser-Part" "" (at 58.42 83.82 0)
-      (effects (font (size 1.27 1.27)) hide)
-    )
-    (property "Notes" "" (at 58.42 83.82 0)
-      (effects (font (size 1.27 1.27)) hide)
-    )
+    (property "Mouser-Part" "571-5645169-4" (at 58.42 83.82 0)
+      (effects (font (size 1.27 1.27)) hide)
+    )
+    (property "Notes" "eBay" (at 58.42 83.82 0)
+      (effects (font (size 1.27 1.27)) hide)
+    )
+    (property "Socket-Mouser" "" (at 58.42 83.82 0)
+      (effects (font (size 1.27 1.27)) hide)
+    )
